Commit message: port to ros2, adding gazebo sim launch package, adding serial port comm controller

File: mini_servo_model/urdf/mini_servo.gazebo.xacro (robot description, xacro)
@@ -2,11 +2,4 @@
 <robot xmlns:xacro="http://www.ros.org/wiki/xacro">
   <xacro:macro name="mini_servo_gazebo" params="robot_name">
-    <!-- Load Gazebo lib and set the robot namespace -->
-    <gazebo>
-      <plugin name="gazebo_ros_control" filename="libgazebo_ros_control.so">
-        <robotNamespace>/${robot_name}</robotNamespace>
-      </plugin>
-    </gazebo>
-    <!-- Link0 -->
     <gazebo reference="${robot_name}_link_0">
       <material>Gazebo/Grey</material>
@@ -14,5 +7,4 @@
       <mu2>0.2</mu2>
     </gazebo>
-    <!-- Link1 -->
     <gazebo reference="${robot_name}_link_1">
       <material>Gazebo/Orange</material>
@@ -20,5 +12,4 @@
       <mu2>0.2</mu2>
     </gazebo>
-    <!-- Link2 -->
     <gazebo reference="${robot_name}_link_2">
       <material>Gazebo/Orange</material>
@@ -26,5 +17,4 @@
       <mu2>0.2</mu2>
     </gazebo>
-    <!-- Link3 -->
     <gazebo reference="${robot_name}_link_3">
       <material>Gazebo/Orange</material>
@@ -32,5 +22,4 @@
       <mu2>0.2</mu2>
     </gazebo>
-    <!-- Link4 -->
     <gazebo reference="${robot_name}_link_4">
       <material>Gazebo/Orange</material>
@@ -38,5 +27,4 @@
       <mu2>0.2</mu2>
     </gazebo>
-    <!-- Link5 -->
     <gazebo reference="${robot_name}_link_5">
       <material>Gazebo/Orange</material>
@@ -44,5 +32,4 @@
       <mu2>0.2</mu2>
     </gazebo>
-    <!-- Link6 -->
     <gazebo reference="${robot_name}_link_6">
       <material>Gazebo/Orange</material>
@@ -50,10 +37,4 @@
       <mu2>0.2</mu2>
     </gazebo>
-    <!-- Link7 -->
-    <gazebo reference="${robot_name}_link_7">
-      <material>Gazebo/Grey</material>
-      <mu1>0.2</mu1>
-      <mu2>0.2</mu2>
-    </gazebo>
   </xacro:macro>
 </robot>

File: mini_servo_model/urdf/mini_servo.urdf.xacro (robot description, xacro)
@@ -1,18 +1,34 @@
 <?xml version="1.0"?>
 <robot name="mini_servo" xmlns:xacro="http://www.ros.org/wiki/xacro">
-  <!-- Import Rviz colors -->
+  <!-- Import RViz colors -->
   <xacro:include filename="$(find mini_servo_model)/urdf/materials.xacro" />
-  <!--Import the mini_servo macro -->
+  <!-- Import the mini_servo macro -->
   <xacro:include filename="$(find mini_servo_model)/urdf/mini_servo.xacro"/>
-  <!--Parameters -->
-  <xacro:arg name="hardware_interface" default="PositionJointInterface"/>
+  <xacro:arg name="ros2_control_hardware_type" default="mock_components"/>
+  <xacro:arg name="use_gazebo" default="false"/>
+  <xacro:arg name="gazebo_controllers_file" default=""/>
+  <xacro:arg name="serial_port" default="/dev/ttyUSB0"/>
+  <xacro:arg name="baud_rate" default="500000"/>
   <xacro:arg name="robot_name" default="mini_servo"/>
   <xacro:arg name="origin_xyz" default="0 0 0"/>
   <xacro:arg name="origin_rpy" default="0 0 0"/>
-  <!-- Fix to world, change if mounted to something -->
+  <!-- Fix to world; change if mounted to something else -->
   <link name="world"/>
-  <!--mini_servo robot-->
-  <xacro:mini_servo hardware_interface="$(arg hardware_interface)" robot_name="$(arg robot_name)" parent="world">
+  <xacro:mini_servo
+      robot_name="$(arg robot_name)"
+      parent="world"
+      ros2_control_hardware_type="$(arg ros2_control_hardware_type)"
+      serial_port="$(arg serial_port)"
+      baud_rate="$(arg baud_rate)">
     <origin xyz="$(arg origin_xyz)" rpy="$(arg origin_rpy)" />
   </xacro:mini_servo>
+  <xacro:if value="$(arg use_gazebo)">
+    <gazebo>
+      <plugin filename="libgz_ros2_control-system.so" name="gz_ros2_control::GazeboSimROS2ControlPlugin">
+        <parameters>$(arg gazebo_controllers_file)</parameters>
+        <hold_joints>true</hold_joints>
+        <position_proportional_gain>25.0</position_proportional_gain>
+      </plugin>
+    </gazebo>
+  </xacro:if>
 </robot>

File: mini_servo_model/urdf/mini_servo.xacro (robot description, xacro)
@@ -3,6 +3,6 @@
   <!-- Import all Gazebo-customization elements, including Gazebo colors -->
   <xacro:include filename="$(find mini_servo_model)/urdf/mini_servo.gazebo.xacro" />
-  <!-- Import Transmissions -->
-  <xacro:include filename="$(find mini_servo_model)/urdf/mini_servo.transmission.xacro" />
+  <!-- Import ros2_control hardware interfaces -->
+  <xacro:include filename="$(find mini_servo_model)/urdf/mini_servo.ros2_control.xacro" />
   <!-- Include Utilities -->
   <xacro:include filename="$(find mini_servo_model)/urdf/utilities.xacro" />
@@ -13,5 +13,5 @@
   <xacro:property name="max_effort" value="300"/>
   <xacro:property name="max_velocity" value="10"/>
-  <xacro:macro name="mini_servo" params="parent hardware_interface robot_name *origin">
+  <xacro:macro name="mini_servo" params="parent robot_name ros2_control_hardware_type:=mock_components serial_port:=/dev/ttyUSB0 baud_rate:=500000 *origin">
     <!--joint between {parent} and link_0-->
     <joint name="${parent}_${robot_name}_joint" type="fixed">
@@ -266,5 +266,9 @@
     <!--Extensions -->
     <xacro:mini_servo_gazebo robot_name="${robot_name}" />
-    <xacro:mini_servo_transmission hardware_interface="${hardware_interface}"/>
+    <xacro:mini_servo_ros2_control
+        robot_name="${robot_name}"
+        ros2_control_hardware_type="${ros2_control_hardware_type}"
+        serial_port="${serial_port}"
+        baud_rate="${baud_rate}"/>
   </xacro:macro>
 </robot>
